Commit message: Added pose goal support to commander, cleaned up misc code

File: urdf/panda.urdf.xacro (robot description, xacro)
@@ -8,6 +8,5 @@
                       >
   </xacro:franka_robot>
-  <link name="left_wall">
-    <!-- left -->
+<!--   <link name="left_wall">
     <visual>
       <geometry>
@@ -38,5 +37,5 @@
       </geometry>
     </collision>
-  </link>
+  </link> -->
   <link name="table">
     <visual>
@@ -58,5 +57,5 @@
      <child  link="$(arg arm_id)_link0" />
   </joint>
-  <joint name="world_to_left_wall" type="fixed">
+ <!--  <joint name="world_to_left_wall" type="fixed">
      <parent link="world"/>
      <child  link="left_wall" />
@@ -67,5 +66,5 @@
      <child  link="rear_wall" />
      <origin xyz="-0.20 0.0 0.5"/>
-  </joint>
+  </joint> -->
   <joint name="world_to_table" type="fixed">
      <parent link="world"/>

Commit message: server removed from launch

File: urdf/panda.urdf.xacro (robot description, xacro)
@@ -57,14 +57,24 @@
      <child  link="$(arg arm_id)_link0" />
   </joint>
- <!--  <joint name="world_to_left_wall" type="fixed">
-     <parent link="world"/>
-     <child  link="left_wall" />
-     <origin xyz="0.30 0.30 0.5"/>
+  <link name="stick">
+    <visual>
+      <geometry>
+        <box size="0.2 0.025 0.025"/>
+      </geometry>
+      <material name="blue">
+        <color rgba="0 0 .8 1"/>
+      </material>
+    </visual>
+    <collision>
+      <geometry>
+        <box size="0.18 0.025 0.025"/>
+      </geometry>
+    </collision>
+  </link>
+  <joint name="panda_hand_to_stick" type="fixed">
+     <parent link="panda_hand"/>
+     <child  link="stick" />
+     <origin xyz="0.12 0 0.12"/>
   </joint>
-    <joint name="world_to_rear_wall" type="fixed">
-     <parent link="world"/>
-     <child  link="rear_wall" />
-     <origin xyz="-0.20 0.0 0.5"/>
-  </joint> -->
   <joint name="world_to_table" type="fixed">
      <parent link="world"/>
@@ -72,3 +82,5 @@
      <origin xyz="0 0 -0.025"/>
   </joint>
+  <disable_collisions link1="stick" link2="panda_leftfinger"/>
+  <disable_collisions link1="stick" link2="panda_rightfinger"/>
 </robot>

Commit message: ease of use for other users

File: urdf/panda.urdf.xacro (robot description, xacro)
@@ -72,4 +72,19 @@
     </collision>
   </link>
+  <link name="camera">
+    <visual>
+      <geometry>
+        <box size="0.5 0.2 1"/>
+      </geometry>
+      <material name="blue_2">
+        <color rgba="0 0 .8 0.1"/>
+      </material>
+    </visual>
+    <collision>
+      <geometry>
+        <box size="0.5 0.2 1"/>
+      </geometry>
+    </collision>
+  </link>
   <joint name="panda_hand_to_stick" type="fixed">
      <parent link="panda_hand"/>
@@ -82,4 +97,9 @@
      <origin xyz="0 0 -0.025"/>
   </joint>
+  <joint name="world_to_camera" type="fixed">
+     <parent link="world"/>
+     <child  link="camera" />
+     <origin xyz="0.45 -0.4 0"/>
+  </joint>
   <disable_collisions link1="stick" link2="panda_leftfinger"/>
   <disable_collisions link1="stick" link2="panda_rightfinger"/>

Commit message: removed interactive audio functionality

File: urdf/panda.urdf.xacro (robot description, xacro)
@@ -57,5 +57,5 @@
      <child  link="$(arg arm_id)_link0" />
   </joint>
-  <link name="stick">
+  <!-- <link name="stick">
     <visual>
       <geometry>
@@ -86,10 +86,10 @@
       </geometry>
     </collision>
-  </link>
-  <joint name="panda_hand_to_stick" type="fixed">
+  </link> -->
+<!--   <joint name="panda_hand_to_stick" type="fixed">
      <parent link="panda_hand"/>
      <child  link="stick" />
      <origin xyz="0.12 0 0.12"/>
-  </joint>
+  </joint> -->
   <joint name="world_to_table" type="fixed">
      <parent link="world"/>
@@ -97,9 +97,9 @@
      <origin xyz="0 0 -0.025"/>
   </joint>
-  <joint name="world_to_camera" type="fixed">
+<!--   <joint name="world_to_camera" type="fixed">
      <parent link="world"/>
      <child  link="camera" />
      <origin xyz="0.45 -0.4 0"/>
-  </joint>
+  </joint> -->
   <disable_collisions link1="stick" link2="panda_leftfinger"/>
   <disable_collisions link1="stick" link2="panda_rightfinger"/>

Commit message: Modified joint_limits and panda urdf to improve

File: urdf/panda.urdf.xacro (robot description, xacro)
@@ -1,12 +1,12 @@
 <?xml version='1.0' encoding='utf-8'?>
 <robot xmlns:xacro="http://www.ros.org/wiki/xacro" name="panda">
-  <xacro:include filename="$(find franka_description)/robots/common/franka_robot.xacro"/>
+  <xacro:include filename="$(find franka_description)/robots/common/franka_robot.xacro" />
   <xacro:arg name="arm_id" default="panda" />
   <link name="world" />
   <xacro:franka_robot arm_id="$(arg arm_id)"
-                      joint_limits="${xacro.load_yaml('$(find franka_description)/robots/panda/joint_limits.yaml')}"
-                      >
+    joint_limits="${xacro.load_yaml('$(find franka_description)/robots/panda/joint_limits.yaml')}"
+  >
   </xacro:franka_robot>
-<!--   <link name="left_wall">
+  <!--   <link name="left_wall">
     <visual>
       <geometry>
@@ -38,69 +38,224 @@
     </collision>
   </link> -->
+<!--
   <link name="table">
     <visual>
       <geometry>
-        <box size="2 1 0.025 "/>
+        <box size="2 1 0.025 " />
       </geometry>
       <material name="blue">
-        <color rgba="0 0 .8 1"/>
-      </material>
-    </visual>
-    <collision>
-      <geometry>
-        <box size="2 1 0.025"/>
-      </geometry>
-    </collision>
-  </link>
+        <color rgba="0 0 .8 1" />
+      </material>
+    </visual>
+    <collision>
+      <geometry>
+        <box size="2 1 0.025" />
+      </geometry>
+    </collision>
+  </link> -->
   <joint name="world_to_link0" type="fixed">
-     <parent link="world"/>
-     <child  link="$(arg arm_id)_link0" />
-  </joint>
-  <!-- <link name="stick">
-    <visual>
-      <geometry>
-        <box size="0.2 0.025 0.025"/>
-      </geometry>
-      <material name="blue">
-        <color rgba="0 0 .8 1"/>
-      </material>
-    </visual>
-    <collision>
-      <geometry>
-        <box size="0.18 0.025 0.025"/>
-      </geometry>
-    </collision>
-  </link>
-  <link name="camera">
-    <visual>
-      <geometry>
-        <box size="0.5 0.2 1"/>
+    <parent link="world" />
+    <child link="$(arg arm_id)_link0" />
+  </joint>
+  <link name="stick">
+    <visual>
+      <geometry>
+        <box size="0.175 0.025 0.025" />
+      </geometry>
+      <material name="blue_3">
+        <color rgba="0 0 .8 0.5" />
+      </material>
+    </visual>
+    <collision>
+      <geometry>
+        <box size="0.175 0.025 0.025" />
+      </geometry>
+    </collision>
+  </link>
+  <!-- <link name="obstacle1">
+    <visual>
+      <geometry>
+        <box size="0.5 0.2 1.5" />
       </geometry>
       <material name="blue_2">
-        <color rgba="0 0 .8 0.1"/>
-      </material>
-    </visual>
-    <collision>
-      <geometry>
-        <box size="0.5 0.2 1"/>
+        <color rgba="0 0 .8 0.1" />
+      </material>
+    </visual>
+    <collision>
+      <geometry>
+        <box size="0.5 0.2 1.5" />
+      </geometry>
+    </collision>
+  </link>
+  <link name="obstacle2">
+    <visual>
+      <geometry>
+        <box size="0.2 0.5 1.5" />
+      </geometry>
+      <material name="blue_2">
+        <color rgba="0 0 .8 0.1" />
+      </material>
+    </visual>
+    <collision>
+      <geometry>
+        <box size="0.2 0.5 1.5" />
       </geometry>
     </collision>
   </link> -->
-<!--   <joint name="panda_hand_to_stick" type="fixed">
-     <parent link="panda_hand"/>
-     <child  link="stick" />
-     <origin xyz="0.12 0 0.12"/>
+  <joint name="panda_hand_to_stick" type="fixed">
+    <parent link="panda_hand" />
+    <child link="stick" />
+    <origin xyz="0.11 0.03 0.12" rpy="0 0 0.4" />
+  </joint>
+  <!-- <joint name="world_to_table" type="fixed">
+    <parent link="world" />
+    <child link="table" />
+    <origin xyz="0 0 -0.005" />
   </joint> -->
-  <joint name="world_to_table" type="fixed">
-     <parent link="world"/>
-     <child  link="table" />
-     <origin xyz="0 0 -0.025"/>
-  </joint>
-<!--   <joint name="world_to_camera" type="fixed">
-     <parent link="world"/>
-     <child  link="camera" />
-     <origin xyz="0.45 -0.4 0"/>
+  <!-- <joint name="world_to_obstacle1" type="fixed">
+    <parent link="world" />
+    <child link="obstacle1" />
+    <origin xyz="0.45 -0.45 0" />
+  </joint>
+  <joint name="world_to_obstacle2" type="fixed">
+    <parent link="world" />
+    <child link="obstacle2" />
+    <origin xyz="0.83 0 0" />
   </joint> -->
-  <disable_collisions link1="stick" link2="panda_leftfinger"/>
-  <disable_collisions link1="stick" link2="panda_rightfinger"/>
+  <disable_collisions link1="stick" link2="panda_leftfinger" />
+  <disable_collisions link1="stick" link2="panda_rightfinger" />
+  <link name="panda_grasptarget">
+    <inertial>
+      <origin rpy="0 0 0" xyz="0 0 0" />
+      <mass value="0.0" />
+      <inertia ixx="0.1" ixy="0" ixz="0" iyy="0.1" iyz="0" izz="0.1" />
+    </inertial>
+    <visual>
+      <origin rpy="0 0 0" xyz="0 0 0" />
+      <geometry>
+        <sphere radius="0.01" />
+      </geometry>
+      <material name="site">
+        <color rgba="1.0 0. 0. 1.0" />
+      </material>
+    </visual>
+  </link>
+  <joint name="panda_grasptarget_hand" type="fixed">
+    <parent link="panda_hand" />
+    <child link="panda_grasptarget" />
+    <origin rpy="0 0 0" xyz="0 0 0.105" />
+  </joint>
+  <link name="arm_mount">
+    <inertial>
+      <origin rpy="0 0 0" xyz="0 -0.01 0.02" />
+      <mass value="0.1" />
+      <inertia ixx="0.1" ixy="0" ixz="0" iyy="0.1" iyz="0" izz="0.1" />
+    </inertial>
+    <visual>
+      <origin rpy="0 3.1415926 -1.57" xyz="0 0 0" />
+      <geometry>
+        <mesh filename="file://$(find deoxys_ros)/urdf/meshes/arm_mount.stl" />
+      </geometry>
+      <!-- <material name="panda_white"/> -->
+      <material name="debug_color">
+        <color rgba="0 1.0 1.0 1.0" />
+      </material>
+    </visual>
+  </link>
+  <joint name="panda_hand_arm_mount" type="fixed">
+    <parent link="panda_grasptarget" />
+    <child link="arm_mount" />
+    <!-- <origin rpy="0 3.14159 -1.57" xyz="0.025 0 -0.068"/> -->
+    <origin rpy="0 0 0" xyz="0.025 0 -0.068" />
+  </joint>
+  <link name="marker_mount">
+    <visual>
+      <origin rpy="-1.57 3.1415926 -1.57" xyz="0 0 0" />
+      <geometry>
+        <mesh filename="file://$(find deoxys_ros)/urdf/meshes/marker_mount.stl" />
+      </geometry>
+      <!-- <material name="panda_white"/> -->
+      <material name="debug_marker_color">
+        <color rgba="1.0 0.0 1.0 1.0" />
+      </material>
+    </visual>
+    <collision>
+      <geometry>
+        <box size="0.01 0.07 0.07" />
+      </geometry>
+    </collision>
+  </link>
+  <joint name="panda_hand_marker_mount" type="fixed">
+    <parent link="arm_mount" />
+    <child link="marker_mount" />
+    <origin rpy="0 0 0" xyz="0.01825 0 0.016" />
+  </joint>
+  <link name="finger_attachment">
+    <visual>
+      <origin rpy="0 0 0" xyz="0 0 0" />
+      <geometry>
+        <box size="0.027 0.105 0.01" />
+      </geometry>
+      <material name="blue_3">
+        <color rgba="0 0 .8 0.5" />
+      </material>
+    </visual>
+    <collision>
+      <geometry>
+        <box size="0.027 0.105 0.01" />
+      </geometry>
+    </collision>
+  </link>
+  <joint name="panda_leftfinger_finger_attachment" type="fixed">
+    <parent link="panda_grasptarget" />
+    <child link="finger_attachment" />
+    <origin rpy="0 0 0" xyz="0 0 0.025" />
+  </joint>
+  <xacro:macro name="camera" params="camera_name x y z">
+    <link name="${camera_name}_collider">
+      <visual>
+        <geometry>
+          <box size="0.15 0.15 0.15"/>
+        </geometry>
+        <material name="red">
+          <color rgba="0.8 0.0 0.0 0.5"/>
+        </material>
+      </visual>
+      <collision>
+        <geometry>
+          <box size="0.15 0.15 0.15"/>
+        </geometry>
+      </collision>
+    </link>
+    <!-- Tall thin box -->
+    <link name="${camera_name}_stand">
+      <visual>
+        <geometry>
+          <box size="0.1 0.1 1.0"/>
+        </geometry>
+        <material name="red">
+          <color rgba="0.8 0.0 0.0 0.5"/>
+        </material>
+      </visual>
+      <collision>
+        <geometry>
+          <box size="0.1 0.1 1.0"/>
+        </geometry>
+      </collision>
+    </link>
+    <joint name="${camera_name}_joint" type="fixed">
+      <origin xyz="${x} ${y} ${z}" rpy="0 0 0"/>
+      <parent link="world"/>
+      <child link="${camera_name}_collider"/>
+    </joint>
+    <joint name="${camera_name}_stand_joint" type="fixed">
+      <origin xyz="0 0 -0.5" rpy="0 0 0"/>
+      <parent link="${camera_name}_collider"/>
+      <child link="${camera_name}_stand"/>
+    </joint>
+  </xacro:macro>
+  <!-- 1.0794; -0.0079469; 0.49701 -->
+  <xacro:camera camera_name="camera0" x="1.0794" y="-0.0079469" z="0.49701" />
+  <!-- 0.57881; -0.45396; 0.51466 -->
+  <xacro:camera camera_name="camera1" x="0.57881" y="-0.45396" z="0.51466" />
 </robot>

Commit message: update deadline push

File: urdf/panda.urdf.xacro (robot description, xacro)
@@ -5,5 +5,5 @@
   <link name="world" />
   <xacro:franka_robot arm_id="$(arg arm_id)"
-    joint_limits="${xacro.load_yaml('$(find franka_description)/robots/panda/joint_limits.yaml')}"
+      joint_limits="${xacro.load_yaml('$(find deoxys_ros)/urdf/joint_limits.yaml')}"
   >
   </xacro:franka_robot>
@@ -61,5 +61,5 @@
     <visual>
       <geometry>
-        <box size="0.175 0.025 0.025" />
+        <box size="0.135 0.025 0.025" />
       </geometry>
       <material name="blue_3">
@@ -69,43 +69,46 @@
     <collision>
       <geometry>
-        <box size="0.175 0.025 0.025" />
-      </geometry>
-    </collision>
-  </link>
-  <!-- <link name="obstacle1">
-    <visual>
-      <geometry>
-        <box size="0.5 0.2 1.5" />
-      </geometry>
-      <material name="blue_2">
-        <color rgba="0 0 .8 0.1" />
-      </material>
-    </visual>
-    <collision>
-      <geometry>
-        <box size="0.5 0.2 1.5" />
-      </geometry>
-    </collision>
-  </link>
-  <link name="obstacle2">
-    <visual>
-      <geometry>
-        <box size="0.2 0.5 1.5" />
-      </geometry>
-      <material name="blue_2">
-        <color rgba="0 0 .8 0.1" />
-      </material>
-    </visual>
-    <collision>
-      <geometry>
-        <box size="0.2 0.5 1.5" />
-      </geometry>
-    </collision>
-  </link> -->
+        <box size="0.135 0.025 0.025" />
+      </geometry>
+    </collision>
+  </link>
   <joint name="panda_hand_to_stick" type="fixed">
     <parent link="panda_hand" />
     <child link="stick" />
-    <origin xyz="0.11 0.03 0.12" rpy="0 0 0.4" />
-  </joint>
+    <!-- Lever -->
+    <!-- <origin xyz="0.11 0.03 0.12" rpy="0 0 0.4" /> -->
+    <!-- Stinger -->
+    <origin xyz="0.10 0.0 0.12" rpy="0 0 0" />
+  </joint>
+  <!-- <link name="obstacle1">
+    <visual>
+      <geometry>
+        <box size="0.5 0.2 1.5" />
+      </geometry>
+      <material name="blue_2">
+        <color rgba="0 0 .8 0.1" />
+      </material>
+    </visual>
+    <collision>
+      <geometry>
+        <box size="0.5 0.2 1.5" />
+      </geometry>
+    </collision>
+  </link>
+  <link name="obstacle2">
+    <visual>
+      <geometry>
+        <box size="0.2 0.5 1.5" />
+      </geometry>
+      <material name="blue_2">
+        <color rgba="0 0 .8 0.1" />
+      </material>
+    </visual>
+    <collision>
+      <geometry>
+        <box size="0.2 0.5 1.5" />
+      </geometry>
+    </collision>
+  </link> -->
   <!-- <joint name="world_to_table" type="fixed">
     <parent link="world" />
@@ -125,4 +128,6 @@
   <disable_collisions link1="stick" link2="panda_leftfinger" />
   <disable_collisions link1="stick" link2="panda_rightfinger" />
+  <disable_collisions link1="finger_attachment" link2="panda_rightfinger" />
+  <disable_collisions link1="finger_attachment" link2="panda_leftfinger" />
   <link name="panda_grasptarget">
     <inertial>
@@ -195,5 +200,8 @@
       <origin rpy="0 0 0" xyz="0 0 0" />
       <geometry>
-        <box size="0.027 0.105 0.01" />
+        <!-- Lever -->
+        <!-- <box size="0.027 0.105 0.01" /> -->
+        <!-- Stinger -->
+        <box size="0.125 0.125 0.045" />
       </geometry>
       <material name="blue_3">
@@ -203,5 +211,5 @@
     <collision>
       <geometry>
-        <box size="0.027 0.105 0.01" />
+        <box size="0.125 0.125 0.045" />
       </geometry>
     </collision>
@@ -210,5 +218,8 @@
     <parent link="panda_grasptarget" />
     <child link="finger_attachment" />
-    <origin rpy="0 0 0" xyz="0 0 0.025" />
+    <!-- Lever -->
+    <!-- <origin rpy="0 0 0" xyz="0 0 0.025" /> -->
+    <!-- Stinger -->
+    <origin rpy="0 0 0" xyz="-0.09 0 0.001" />
   </joint>
   <xacro:macro name="camera" params="camera_name x y z">
@@ -255,7 +266,33 @@
     </joint>
   </xacro:macro>
+  <xacro:macro name="obstacle" params="obstacle_name x y z l w h">
+    <link name="${obstacle_name}">
+      <visual>
+        <geometry>
+          <box size="${l} ${w} ${h}" />
+        </geometry>
+        <material name="blue_2">
+          <color rgba="0 0 .8 0.1" />
+        </material>
+      </visual>
+      <collision>
+        <geometry>
+          <box size="${l} ${w} ${h}" />
+        </geometry>
+      </collision>
+    </link>
+    <joint name="world_to_${obstacle_name}" type="fixed">
+      <parent link="world" />
+      <child link="${obstacle_name}" />
+      <origin xyz="${x} ${y} ${z}" />
+    </joint>
+  </xacro:macro>
   <!-- 1.0794; -0.0079469; 0.49701 -->
-  <xacro:camera camera_name="camera0" x="1.0794" y="-0.0079469" z="0.49701" />
+  <xacro:camera camera_name="camera0" x="0.52753" y="-0.56482" z="0.51105"  />
   <!-- 0.57881; -0.45396; 0.51466 -->
-  <xacro:camera camera_name="camera1" x="0.57881" y="-0.45396" z="0.51466" />
+  <!-- <xacro:camera camera_name="camera1" x="0.57881" y="-0.45396" z="0.51466" /> -->
+  <xacro:obstacle obstacle_name="rear_wall" x="-0.4" y="0" z="0.5" l="0.1" w="2.0" h="2.0"/>
+  <xacro:obstacle obstacle_name="ceiling" x="1.0" y="0" z="1.25" l="2.5" w="3.0" h="0.1"/>
+  <xacro:obstacle obstacle_name="left_wall" x="1.0" y="0.5" z="0.5" l="2.0" w="0.1" h="2.0"/>
+  <xacro:obstacle obstacle_name="light_stand" x="-0.1" y="-0.6" z="0.5" l="0.1" w="0.1" h="1.0"/>
 </robot>

Commit message: server osc move

File: urdf/panda.urdf.xacro (robot description, xacro)
@@ -61,5 +61,5 @@
     <visual>
       <geometry>
-        <box size="0.135 0.025 0.025" />
+        <box size="0.13 0.025 0.025" />
       </geometry>
       <material name="blue_3">
@@ -69,5 +69,5 @@
     <collision>
       <geometry>
-        <box size="0.135 0.025 0.025" />
+        <box size="0.13 0.025 0.025" />
       </geometry>
     </collision>
@@ -79,5 +79,5 @@
     <!-- <origin xyz="0.11 0.03 0.12" rpy="0 0 0.4" /> -->
     <!-- Stinger -->
-    <origin xyz="0.10 0.0 0.12" rpy="0 0 0" />
+    <origin xyz="0.115 0.0 0.11" rpy="0 0 0" />
   </joint>
   <!-- <link name="obstacle1">

Commit message: deadline dump 2/21

File: urdf/panda.urdf.xacro (robot description, xacro)
@@ -61,5 +61,5 @@
     <visual>
       <geometry>
-        <box size="0.13 0.025 0.025" />
+        <box size="0.15 0.025 0.025" />
       </geometry>
       <material name="blue_3">
